Commit message: Split link7 into motor and link

File: urdf/ee/openarm_hand_macro.xacro (robot description, xacro)
@@ -25,4 +25,7 @@
         <xacro:openarm-ee-kinematics-link config="${ee_kinematics_link}" name="${name}" />
         <geometry>
+          <mesh filename="package://${description_pkg}/meshes/ee/${ee_type}/visual/motor8.dae" scale="0.001 0.001 0.001" />
+        </geometry>
+        <geometry>
           <mesh filename="package://${description_pkg}/meshes/ee/${ee_type}/visual/${name}.dae" scale="0.001 0.001 0.001" />
         </geometry>

File: urdf/robot/v10.urdf.xacro (robot description, xacro)
@@ -7,5 +7,5 @@
   <xacro:arg name="has_head" default="false" />
   <xacro:arg name="no_prefix" default="false"/>
-  <xacro:arg name="hand" default="true" />
+  <xacro:arg name="hand" default="false" />
   <xacro:if value="$(eval ee_type == 'none')">
     <xacro:property name="hand" value="false"/>
