Commit message: Enable ros2_control head module

File: urdf/robot/openarm_robot.xacro (robot description, xacro)
@@ -18,4 +18,5 @@
             hand:='false'
             ee_type:=''
+            has_head
             ros2_control:=false
             use_fake_hardware:=false
@@ -26,5 +27,5 @@
             arm_connected_to='base'
             body_connected_to='world'
-            bimanual:=false
+            bimanual
             right_arm_base_xyz='0 0 0'
             left_arm_base_xyz='0 0 0'
@@ -97,5 +98,6 @@
             left_arm_prefix="${left_arm_prefix}"
             right_arm_prefix="${right_arm_prefix}"
-            hand="${hand}"/>
+            hand="${hand}"
+            has_head="${has_head}"/>
         </xacro:if>
         <xacro:if value="$(eval hand and ee_type == 'openarm_hand')">

File: urdf/robot/v10.urdf.xacro (robot description, xacro)
@@ -5,4 +5,5 @@
   <xacro:arg name="body_type" default="v10" />
   <xacro:arg name="ee_type" default="openarm_hand" />
+  <xacro:arg name="has_head" default="false" />
   <xacro:arg name="no_prefix" default="false"/>
   <xacro:arg name="hand" default="true" />
@@ -18,5 +19,5 @@
   <xacro:arg name="use_fake_hardware" default="false" />
   <xacro:arg name="fake_sensor_commands" default="false" />
-  <xacro:arg name="bimanual" default="false" />
+  <xacro:arg name="bimanual" default="true" />
   <xacro:arg name="right_arm_base_xyz" default="0.0 -0.031 0.698" />
   <xacro:arg name="right_arm_base_rpy" default="1.5708 0 0" />
@@ -38,4 +39,5 @@
   hand="$(arg hand)"
   ee_type="$(arg ee_type)"
+  has_head="$(arg has_head)"
   ros2_control="$(arg ros2_control)"
   left_arm_prefix="$(arg left_arm_prefix)"

File: urdf/ros2_control/openarm.bimanual.ros2_control.xacro (robot description, xacro)
@@ -6,4 +6,5 @@
              fake_sensor_commands:=^|false
              hand:=^|false
+             has_head
              left_arm_prefix:=^|left_
              right_arm_prefix:=^|right_
@@ -79,4 +80,23 @@
       </xacro:if>
     </ros2_control>
+    <!-- Head Module Hardware Interface -->
+    <xacro:if value="${has_head}">
+      <ros2_control name="openarm_head" type="system">
+        <hardware>
+          <plugin>openarm_hardware/OpenArmHeadV1</plugin>
+          <param name="can_fd">${can_fd}</param>
+        </hardware>
+        <joint name="openarm_head_pitch">
+          <command_interface name="position"/>
+          <state_interface name="position"/>
+          <state_interface name="velocity"/>
+        </joint>
+        <joint name="openarm_head_yaw">
+          <command_interface name="position"/>
+          <state_interface name="position"/>
+          <state_interface name="velocity"/>
+        </joint>
+      </ros2_control>
+    </xacro:if>
   </xacro:macro>
 </robot>

Commit message: Head module vis

File: urdf/robot/openarm_robot.xacro (robot description, xacro)
@@ -51,6 +51,10 @@
         <xacro:include filename="$(find openarm_description)/urdf/ee/${ee_type}_arguments.xacro" />
     </xacro:if>
+    <xacro:if value="${has_head}">
+        <xacro:include filename="$(find openarm_description)/urdf/head/openarm_head.xacro" />
+    </xacro:if>
     <xacro:property name="arm_prefix_modified" value="${'' if arm_prefix == '' else arm_prefix + '_'}" />
     <xacro:property name="body_prefix_modified" value="${'' if body_prefix == '' else body_prefix + '_'}" />
+    <xacro:property name="body_link0_name" value="${'body_link0' if no_prefix else 'openarm_body_link0'}" />
     <xacro:if value="${bimanual}">
         <xacro:openarm_body
@@ -65,4 +69,11 @@
         kinematics="${body_kinematics}"
         kinematics_link="${body_kinematics_link}" />
+        <xacro:if value="${has_head}">
+            <joint name="openarm_head_mount" type="fixed">
+                <parent link="${body_link0_name}" />
+                <child link="base_link" />
+                <origin xyz="-0.0025 0 0.750" rpy="0 0 -1.5708" />
+            </joint>
+        </xacro:if>
         <!-- left arm -->
         <xacro:openarm_arm
@@ -104,5 +115,5 @@
             right_arm_prefix="${right_arm_prefix}"
             hand="${hand}"
-            has_head="${has_head}"/>
+            has_head="${has_head_enabled}"/>
         </xacro:if>
         <xacro:if value="$(eval hand and ee_type == 'openarm_hand')">

File: urdf/robot/v10.urdf.xacro (robot description, xacro)
@@ -5,5 +5,5 @@
   <xacro:arg name="body_type" default="v10" />
   <xacro:arg name="ee_type" default="openarm_hand" />
-  <xacro:arg name="has_head" default="false" />
+  <xacro:arg name="has_head" default="true" />
   <xacro:arg name="no_prefix" default="false"/>
   <xacro:arg name="hand" default="false" />

Commit message: Add RH56F1 option as end-effector

File: urdf/robot/openarm_robot.xacro (robot description, xacro)
@@ -16,6 +16,5 @@
             xyz:='0 0 0'
             rpy:='0 0 0'
-            hand:='false'
-            ee_type:=''
+            ee_type
             has_head
             ros2_control:=false
@@ -44,13 +43,10 @@
     <xacro:include filename="$(find openarm_description)/urdf/body/openarm_body_macro.xacro" />
     <xacro:include filename="$(find openarm_description)/urdf/body/openarm_body.xacro" />
-    <xacro:include filename="$(find openarm_description)/urdf/ee/openarm_hand.xacro" />
-    <xacro:include filename="$(find openarm_description)/urdf/ee/openarm_hand_macro.xacro" />
     <xacro:include filename="$(find openarm_description)/urdf/ros2_control/openarm.ros2_control.xacro" />
     <xacro:include filename="$(find openarm_description)/urdf/ros2_control/openarm.bimanual.ros2_control.xacro" />
-    <xacro:if value="${ee_type != 'none'}">
-        <xacro:include filename="$(find openarm_description)/urdf/ee/${ee_type}_arguments.xacro" />
-    </xacro:if>
-    <xacro:if value="${has_head}">
-        <xacro:include filename="$(find openarm_description)/urdf/head/openarm_head.xacro" />
+    <xacro:if value="${ee_type == 'openarm_hand'}">
+        <xacro:include filename="$(find openarm_description)/urdf/ee/openarm_hand.xacro" />
+        <xacro:include filename="$(find openarm_description)/urdf/ee/openarm_hand_macro.xacro" />
+        <xacro:include filename="$(find openarm_description)/urdf/ee/openarm_hand_arguments.xacro" />
     </xacro:if>
     <xacro:property name="arm_prefix_modified" value="${'' if arm_prefix == '' else arm_prefix + '_'}" />
@@ -70,4 +66,5 @@
         kinematics_link="${body_kinematics_link}" />
         <xacro:if value="${has_head}">
+            <xacro:include filename="$(find openarm_description)/urdf/head/openarm_head.xacro" />
             <joint name="openarm_head_mount" type="fixed">
                 <parent link="${body_link0_name}" />
@@ -117,5 +114,5 @@
             has_head="${has_head}"/>
         </xacro:if>
-        <xacro:if value="$(eval hand and ee_type == 'openarm_hand')">
+        <xacro:if value="${ee_type == 'openarm_hand'}">
             <xacro:openarm_hand
                 connected_to="openarm_left_link7"
@@ -144,5 +141,47 @@
                 description_pkg="$(arg description_pkg)"
             />
-          </xacro:if>
+        </xacro:if>
+        <xacro:if value="${ee_type == 'rh56f1'}">
+            <link name="left_hand_mount" type="fixed">
+                <visual>
+                    <origin rpy="0 0 3.1416" xyz="0 0 0"/>
+                    <geometry>
+                    <mesh filename="package://openarm_description/meshes/ee/rh56f1/visual/rh56f1_mount.stl" scale="0.001 0.001 0.001"/>
+                    </geometry>
+                </visual>
+            </link>
+            <xacro:include filename="$(find inspire_hand_description)/RH56F1/left/urdf/RH56F1_L.xacro" />
+            <xacro:RH56F1_L />
+            <joint name="left_arm_to_mount" type="fixed">
+                <parent link="openarm_left_link7" />
+                <child link="left_hand_mount" />
+                <origin xyz="0 0 0.0495" rpy="0 0 0" />
+            </joint>
+            <joint name="left_mount_to_rh56f1" type="fixed">
+                <parent link="left_hand_mount" />
+                <child link="left_hand_base_link" />
+                <origin xyz="0 0 0.006" rpy="0 0 1.5708" />
+            </joint>
+            <link name="right_hand_mount" type="fixed">
+                <visual>
+                    <origin rpy="0 0 0" xyz="0 0 0"/>
+                    <geometry>
+                    <mesh filename="package://openarm_description/meshes/ee/rh56f1/visual/rh56f1_mount.stl" scale="0.001 0.001 0.001"/>
+                    </geometry>
+                </visual>
+            </link>
+            <xacro:include filename="$(find inspire_hand_description)/RH56F1/right/urdf/RH56F1_R.xacro" />
+            <xacro:RH56F1_R />
+            <joint name="right_arm_to_mount" type="fixed">
+                <parent link="openarm_right_link7" />
+                <child link="right_hand_mount" />
+                <origin xyz="0 0 0.0495" rpy="0 0 0" />
+            </joint>
+            <joint name="right_mount_to_rh56f1" type="fixed">
+                <parent link="right_hand_mount" />
+                <child link="right_hand_base_link" />
+                <origin xyz="0 0 0.006" rpy="0 0 -1.5708" />
+            </joint>
+        </xacro:if>
     </xacro:if>
     <xacro:if value="${not bimanual}">
@@ -170,9 +209,8 @@
             can_fd="${can_fd}"/>
         </xacro:if>
-        <xacro:if value="${hand and ee_type == 'openarm_hand'}">
+        <xacro:if value="${ee_type == 'openarm_hand'}">
         <xacro:property name="special_connection" value="$(arg special_connection)" />
         <!-- <xacro:property name="connection" value="${special_connection if special_connection != '' else arm_type + '_link7'}" /> -->
         <xacro:property name="connection" value="${special_connection if special_connection != '' else 'openarm' + '_link7'}" />
-        <xacro:if value="$(eval hand and ee_type == 'openarm_hand')">
         <xacro:openarm_hand
             connected_to="${arm_prefix_modified}${connection}"
@@ -188,6 +226,5 @@
             description_pkg="$(arg description_pkg)"/>
         </xacro:if>
-        </xacro:if>
-        </xacro:if>
+    </xacro:if>
   </xacro:macro>
 </robot>

File: urdf/robot/v10.urdf.xacro (robot description, xacro)
@@ -4,11 +4,7 @@
   <xacro:arg name="arm_type" default="v10" />
   <xacro:arg name="body_type" default="v10" />
-  <xacro:arg name="ee_type" default="openarm_hand" />
+  <xacro:arg name="ee_type" default="none" />
   <xacro:arg name="has_head" default="true" />
   <xacro:arg name="no_prefix" default="false"/>
-  <xacro:arg name="hand" default="false" />
-  <xacro:if value="$(eval ee_type == 'none')">
-    <xacro:property name="hand" value="false"/>
-  </xacro:if>
   <xacro:arg name="parent" default="world" />
   <xacro:arg name="xyz" default="0 0 0" />
@@ -40,5 +36,4 @@
   body_kinematics_link="${xacro.load_yaml('$(find openarm_description)/config/body/v10/kinematics.yaml')}"
   ee_kinematics_link="${xacro.load_yaml('$(find openarm_description)/config/hand/openarm_hand/kinematics_link.yaml')}"
-  hand="$(arg hand)"
   ee_type="$(arg ee_type)"
   has_head="$(arg has_head)"
