Commit message: Add xhand1 end-effector support and refactor ee_type path resolution
Co-Authored-By: Claude Opus 4.6 (1M context) <noreply@anthropic.com>

File: urdf/robot/openarm_robot.xacro (robot description, xacro)
@@ -184,4 +184,19 @@
             </joint>
         </xacro:if>
+        <xacro:if value="${ee_type == 'xhand1'}">
+            <xacro:include filename="${xhand_include_prefix}/urdf/xhand1_hand.urdf.xacro" />
+            <xacro:xhand1_hand
+                side="left"
+                reflect="-1"
+                parent_link="openarm_left_link7"
+                origin_xyz="0 0 0.055"
+                origin_rpy="0 0 1.5708" />
+            <xacro:xhand1_hand
+                side="right"
+                reflect="1"
+                parent_link="openarm_right_link7"
+                origin_xyz="0 0 0.055"
+                origin_rpy="0 0 -1.5708" />
+        </xacro:if>
     </xacro:if>
     <xacro:if value="${not bimanual}">

File: urdf/robot/v10.urdf.xacro (robot description, xacro)
@@ -2,20 +2,37 @@
 <robot xmlns:xacro="http://www.ros.org/wiki/xacro" name="openarm">
   <xacro:arg name="standalone" default="false" />
-  <!-- ROS mode (default): use package:// for meshes -->
+  <xacro:arg name="ee_type" default="none" />
+  <!-- Common mesh prefix -->
   <xacro:unless value="$(arg standalone)">
     <xacro:property name="mesh_prefix" value="package://openarm_description" scope="global" />
-    <xacro:property name="hand_mesh_prefix" value="package://inspire_hand_description" scope="global" />
-    <xacro:property name="hand_include_prefix" value="$(find inspire_hand_description)" scope="global" />
   </xacro:unless>
-  <!-- Standalone mode: use relative paths -->
   <xacro:if value="$(arg standalone)">
     <xacro:property name="mesh_prefix" value="." scope="global" />
-    <xacro:property name="hand_mesh_prefix" value="./inspire_hand_description" scope="global" />
-    <xacro:property name="hand_include_prefix" value="../../inspire_hand_description" scope="global" />
+  </xacro:if>
+  <!-- Inspire hand (rh56f1) paths — only resolved when needed -->
+  <xacro:if value="${'$(arg ee_type)' == 'rh56f1'}">
+    <xacro:unless value="$(arg standalone)">
+      <xacro:property name="hand_mesh_prefix" value="package://inspire_hand_description" scope="global" />
+      <xacro:property name="hand_include_prefix" value="$(find inspire_hand_description)" scope="global" />
+    </xacro:unless>
+    <xacro:if value="$(arg standalone)">
+      <xacro:property name="hand_mesh_prefix" value="./inspire_hand_description" scope="global" />
+      <xacro:property name="hand_include_prefix" value="../../inspire_hand_description" scope="global" />
+    </xacro:if>
+  </xacro:if>
+  <!-- xhand1 paths — only resolved when needed -->
+  <xacro:if value="${'$(arg ee_type)' == 'xhand1'}">
+    <xacro:unless value="$(arg standalone)">
+      <xacro:property name="xhand_mesh_prefix" value="package://xhand_description" scope="global" />
+      <xacro:property name="xhand_include_prefix" value="$(find xhand_description)" scope="global" />
+    </xacro:unless>
+    <xacro:if value="$(arg standalone)">
+      <xacro:property name="xhand_mesh_prefix" value="../xhand_description" scope="global" />
+      <xacro:property name="xhand_include_prefix" value="../../../xhand_description" scope="global" />
+    </xacro:if>
   </xacro:if>
   <xacro:include filename="openarm_robot.xacro"/>
   <xacro:arg name="arm_type" default="v10" />
   <xacro:arg name="body_type" default="v10" />
-  <xacro:arg name="ee_type" default="none" />
   <xacro:arg name="has_head" default="true" />
   <xacro:arg name="no_prefix" default="false"/>
