Commit message: absolute path

File: urdf/arm/openarm_arm.xacro (robot description, xacro)
@@ -1,5 +1,5 @@
 <?xml version='1.0' encoding='utf-8'?>
 <robot xmlns:xacro="http://www.ros.org/wiki/xacro" name="openarm">
-  <xacro:include filename="$(find openarm_description)/urdf/arm/openarm_macro.xacro" />
+  <xacro:include filename="${pkg_path}/urdf/arm/openarm_macro.xacro" />
   <xacro:macro name="openarm_arm" params="arm_type arm_prefix:='' no_prefix:=false description_pkg:='openarm_description' connected_to:='base' xyz:='0 0 0' rpy:='0 0 0' joint_limits inertials kinematics kinematics_link kinematics_offset:=none " >
     <xacro:property name="prefix" value="${'' if no_prefix else 'openarm' + '_' + arm_prefix}" />

File: urdf/arm/openarm_macro.xacro (robot description, xacro)
@@ -27,5 +27,5 @@
         <xacro:openarm-kinematics-link config="${kinematics_link}" name="${name}" />
         <geometry>
-          <mesh filename="package://${description_pkg}/meshes/arm/${arm_type}/visual/${name}.dae" scale="0.001 ${0.001*reflect} 0.001" />
+          <mesh filename="${mesh_prefix}/meshes/arm/${arm_type}/visual/${name}.dae" scale="0.001 ${0.001*reflect} 0.001" />
         </geometry>
       </visual>
@@ -33,6 +33,6 @@
         <xacro:openarm-kinematics-link config="${kinematics_link}" name="${name}" />
         <geometry>
-          <mesh filename="package://openarm_description/meshes/arm/${arm_type}/collision/${name}_symp.stl" scale="0.001 ${0.001*reflect} 0.001" />
-          <!-- <mesh filename="package://openarm_description/meshes/arm/${arm_type}/collision/${name}.stl" scale="0.001 0.001 0.001" /> -->
+          <mesh filename="${mesh_prefix}/meshes/arm/${arm_type}/collision/${name}_symp.stl" scale="0.001 ${0.001*reflect} 0.001" />
+          <!-- <mesh filename="${mesh_prefix}/meshes/arm/${arm_type}/collision/${name}.stl" scale="0.001 0.001 0.001" /> -->
         </geometry>
       </collision>

File: urdf/body/openarm_body.xacro (robot description, xacro)
@@ -1,5 +1,5 @@
 <?xml version="1.0" encoding="utf-8"?>
 <robot xmlns:xacro="http://www.ros.org/wiki/xacro" name="openarm_body">
-  <xacro:include filename="$(find openarm_description)/urdf/body/openarm_body_macro.xacro" />
+  <xacro:include filename="${pkg_path}/urdf/body/openarm_body_macro.xacro" />
       <xacro:macro name="openarm_body"
       params="body_type

File: urdf/body/openarm_body_macro.xacro (robot description, xacro)
@@ -23,5 +23,5 @@
         <xacro:openarm-body-kinematics config="${kinematics_link}" name="${name}" />
         <geometry>
-          <mesh filename="package://${description_pkg}/meshes/body/${body_type}/visual/${name}.dae" scale="0.001 0.001 0.001" />
+          <mesh filename="${mesh_prefix}/meshes/body/${body_type}/visual/${name}.dae" scale="0.001 0.001 0.001" />
         </geometry>
       </visual>
@@ -29,6 +29,6 @@
         <xacro:openarm-body-kinematics config="${kinematics_link}" name="${name}" />
         <geometry>
-          <mesh filename="package://openarm_description/meshes/body/${body_type}/collision/${name}_symp.stl" scale="0.001 0.001 0.001" />
-          <!-- <mesh filename="package://openarm_description/meshes/arm/${arm_type}/collision/${name}.stl" scale="0.001 0.001 0.001" /> -->
+          <mesh filename="${mesh_prefix}/meshes/body/${body_type}/collision/${name}_symp.stl" scale="0.001 0.001 0.001" />
+          <!-- <mesh filename="${mesh_prefix}/meshes/arm/${arm_type}/collision/${name}.stl" scale="0.001 0.001 0.001" /> -->
         </geometry>
       </collision>

File: urdf/ee/openarm_hand.xacro (robot description, xacro)
@@ -29,5 +29,5 @@
         <xacro:openarm-ee-kinematics-link config="${ee_kinematics_link}" name="left_finger" />
         <geometry>
-          <mesh filename="package://${description_pkg}/meshes/ee/${ee_type}/visual/finger.dae" scale="0.001 0.001 0.001"/>
+          <mesh filename="${mesh_prefix}/meshes/ee/${ee_type}/visual/finger.dae" scale="0.001 0.001 0.001"/>
         </geometry>
       </visual>
@@ -35,5 +35,5 @@
         <xacro:openarm-ee-kinematics-link config="${ee_kinematics_link}" name="left_finger" />
         <geometry>
-          <mesh filename="package://${description_pkg}/meshes/ee/${ee_type}/collision/finger.stl" scale="0.001 0.001 0.001" />
+          <mesh filename="${mesh_prefix}/meshes/ee/${ee_type}/collision/finger.stl" scale="0.001 0.001 0.001" />
         </geometry>
       </collision>
@@ -44,5 +44,5 @@
         <xacro:openarm-ee-kinematics-link config="${ee_kinematics_link}" name="right_finger" />
         <geometry>
-          <mesh filename="package://${description_pkg}/meshes/ee/${ee_type}/visual/finger.dae" scale="0.001 -0.001 0.001"/>
+          <mesh filename="${mesh_prefix}/meshes/ee/${ee_type}/visual/finger.dae" scale="0.001 -0.001 0.001"/>
         </geometry>
       </visual>
@@ -50,5 +50,5 @@
         <xacro:openarm-ee-kinematics-link config="${ee_kinematics_link}" name="right_finger" />
         <geometry>
-          <mesh filename="package://${description_pkg}/meshes/ee/${ee_type}/collision/finger.stl" scale="0.001 -0.001 0.001" />
+          <mesh filename="${mesh_prefix}/meshes/ee/${ee_type}/collision/finger.stl" scale="0.001 -0.001 0.001" />
         </geometry>
       </collision>

File: urdf/ee/openarm_hand_macro.xacro (robot description, xacro)
@@ -25,8 +25,8 @@
         <xacro:openarm-ee-kinematics-link config="${ee_kinematics_link}" name="${name}" />
         <geometry>
-          <mesh filename="package://${description_pkg}/meshes/ee/${ee_type}/visual/motor8.dae" scale="0.001 0.001 0.001" />
+          <mesh filename="${mesh_prefix}/meshes/ee/${ee_type}/visual/motor8.dae" scale="0.001 0.001 0.001" />
         </geometry>
         <geometry>
-          <mesh filename="package://${description_pkg}/meshes/ee/${ee_type}/visual/${name}.dae" scale="0.001 0.001 0.001" />
+          <mesh filename="${mesh_prefix}/meshes/ee/${ee_type}/visual/${name}.dae" scale="0.001 0.001 0.001" />
         </geometry>
       </visual>
@@ -34,5 +34,5 @@
         <xacro:openarm-ee-kinematics-link config="${ee_kinematics_link}" name="${name}" />
         <geometry>
-          <mesh filename="package://openarm_description/meshes/ee/${ee_type}/collision/${name}.stl" scale="0.001 0.001 0.001" />
+          <mesh filename="${mesh_prefix}/meshes/ee/${ee_type}/collision/${name}.stl" scale="0.001 0.001 0.001" />
         </geometry>
       </collision>

File: urdf/head/openarm_head.xacro (robot description, xacro)
@@ -10,5 +10,5 @@
     <origin xyz="0 0 0" rpy="0 0 0"/>
     <geometry>
-      <mesh filename="package://openarm_description/meshes/head/visual/head_base_link.stl" scale="0.001 0.001 0.001"/>
+      <mesh filename="${mesh_prefix}/meshes/head/visual/head_base_link.stl" scale="0.001 0.001 0.001"/>
     </geometry>
   </visual>
@@ -16,5 +16,5 @@
     <origin xyz="0 0 0" rpy="0 0 0"/>
     <geometry>
-      <mesh filename="package://openarm_description/meshes/head/visual/head_base_link.stl" scale="0.001 0.001 0.001"/>
+      <mesh filename="${mesh_prefix}/meshes/head/visual/head_base_link.stl" scale="0.001 0.001 0.001"/>
     </geometry>
   </collision>
@@ -29,5 +29,5 @@
     <origin xyz="0.0125 0.0 -0.0415" rpy="0 0 0"/>
     <geometry>
-      <mesh filename="package://openarm_description/meshes/head/visual/pitch_motor_rotor_1.stl" scale="0.001 0.001 0.001"/>
+      <mesh filename="${mesh_prefix}/meshes/head/visual/pitch_motor_rotor_1.stl" scale="0.001 0.001 0.001"/>
     </geometry>
   </visual>
@@ -35,5 +35,5 @@
     <origin xyz="0.0125 0.0 -0.0415" rpy="0 0 0"/>
     <geometry>
-      <mesh filename="package://openarm_description/meshes/head/visual/pitch_motor_rotor_1.stl" scale="0.001 0.001 0.001"/>
+      <mesh filename="${mesh_prefix}/meshes/head/visual/pitch_motor_rotor_1.stl" scale="0.001 0.001 0.001"/>
     </geometry>
   </collision>
@@ -48,5 +48,5 @@
     <origin xyz="-0.025 0.001656 -0.060428" rpy="0 0 0"/>
     <geometry>
-      <mesh filename="package://openarm_description/meshes/head/visual/pitch_motor_case_1.stl" scale="0.001 0.001 0.001"/>
+      <mesh filename="${mesh_prefix}/meshes/head/visual/pitch_motor_case_1.stl" scale="0.001 0.001 0.001"/>
     </geometry>
   </visual>
@@ -54,5 +54,5 @@
     <origin xyz="-0.025 0.001656 -0.060428" rpy="0 0 0"/>
     <geometry>
-      <mesh filename="package://openarm_description/meshes/head/visual/pitch_motor_case_1.stl" scale="0.001 0.001 0.001"/>
+      <mesh filename="${mesh_prefix}/meshes/head/visual/pitch_motor_case_1.stl" scale="0.001 0.001 0.001"/>
     </geometry>
   </collision>
@@ -67,5 +67,5 @@
     <origin xyz="0.013435 -0.013435 -0.0785" rpy="0 0 0"/>
     <geometry>
-      <mesh filename="package://openarm_description/meshes/head/visual/pitch_motor_case_2.stl" scale="0.001 0.001 0.001"/>
+      <mesh filename="${mesh_prefix}/meshes/head/visual/pitch_motor_case_2.stl" scale="0.001 0.001 0.001"/>
     </geometry>
   </visual>
@@ -73,5 +73,5 @@
     <origin xyz="0.013435 -0.013435 -0.0785" rpy="0 0 0"/>
     <geometry>
-      <mesh filename="package://openarm_description/meshes/head/visual/pitch_motor_case_2.stl" scale="0.001 0.001 0.001"/>
+      <mesh filename="${mesh_prefix}/meshes/head/visual/pitch_motor_case_2.stl" scale="0.001 0.001 0.001"/>
     </geometry>
   </collision>
@@ -86,5 +86,5 @@
     <origin xyz="0.0 -0.0 -0.116" rpy="0 0 0"/>
     <geometry>
-      <mesh filename="package://openarm_description/meshes/head/visual/pitch_motor_rotor_2.stl" scale="0.001 0.001 0.001"/>
+      <mesh filename="${mesh_prefix}/meshes/head/visual/pitch_motor_rotor_2.stl" scale="0.001 0.001 0.001"/>
     </geometry>
   </visual>
@@ -92,5 +92,5 @@
     <origin xyz="0.0 -0.0 -0.116" rpy="0 0 0"/>
     <geometry>
-      <mesh filename="package://openarm_description/meshes/head/visual/pitch_motor_rotor_2.stl" scale="0.001 0.001 0.001"/>
+      <mesh filename="${mesh_prefix}/meshes/head/visual/pitch_motor_rotor_2.stl" scale="0.001 0.001 0.001"/>
     </geometry>
   </collision>
@@ -105,5 +105,5 @@
     <origin xyz="-0.00675 -0.011691 -0.1245" rpy="0 0 0"/>
     <geometry>
-      <mesh filename="package://openarm_description/meshes/head/visual/Body1_1.stl" scale="0.001 0.001 0.001"/>
+      <mesh filename="${mesh_prefix}/meshes/head/visual/Body1_1.stl" scale="0.001 0.001 0.001"/>
     </geometry>
   </visual>
@@ -111,5 +111,5 @@
     <origin xyz="-0.00675 -0.011691 -0.1245" rpy="0 0 0"/>
     <geometry>
-      <mesh filename="package://openarm_description/meshes/head/visual/Body1_1.stl" scale="0.001 0.001 0.001"/>
+      <mesh filename="${mesh_prefix}/meshes/head/visual/Body1_1.stl" scale="0.001 0.001 0.001"/>
     </geometry>
   </collision>
@@ -124,5 +124,5 @@
     <origin xyz="0.0 -0.047 -0.1295" rpy="0 0 0"/>
     <geometry>
-      <mesh filename="package://openarm_description/meshes/head/visual/camera.stl" scale="0.001 0.001 0.001"/>
+      <mesh filename="${mesh_prefix}/meshes/head/visual/camera.stl" scale="0.001 0.001 0.001"/>
     </geometry>
   </visual>
@@ -130,5 +130,5 @@
     <origin xyz="0.0 -0.047 -0.1295" rpy="0 0 0"/>
     <geometry>
-      <mesh filename="package://openarm_description/meshes/head/visual/camera.stl" scale="0.001 0.001 0.001"/>
+      <mesh filename="${mesh_prefix}/meshes/head/visual/camera.stl" scale="0.001 0.001 0.001"/>
     </geometry>
   </collision>

File: urdf/robot/openarm_robot.xacro (robot description, xacro)
@@ -39,14 +39,14 @@
             "
             >
-    <xacro:include filename="$(find openarm_description)/urdf/arm/openarm_macro.xacro" />
-    <xacro:include filename="$(find openarm_description)/urdf/arm/openarm_arm.xacro" />
-    <xacro:include filename="$(find openarm_description)/urdf/body/openarm_body_macro.xacro" />
-    <xacro:include filename="$(find openarm_description)/urdf/body/openarm_body.xacro" />
-    <xacro:include filename="$(find openarm_description)/urdf/ros2_control/openarm.ros2_control.xacro" />
-    <xacro:include filename="$(find openarm_description)/urdf/ros2_control/openarm.bimanual.ros2_control.xacro" />
+    <xacro:include filename="${pkg_path}/urdf/arm/openarm_macro.xacro" />
+    <xacro:include filename="${pkg_path}/urdf/arm/openarm_arm.xacro" />
+    <xacro:include filename="${pkg_path}/urdf/body/openarm_body_macro.xacro" />
+    <xacro:include filename="${pkg_path}/urdf/body/openarm_body.xacro" />
+    <xacro:include filename="${pkg_path}/urdf/ros2_control/openarm.ros2_control.xacro" />
+    <xacro:include filename="${pkg_path}/urdf/ros2_control/openarm.bimanual.ros2_control.xacro" />
     <xacro:if value="${ee_type == 'openarm_hand'}">
-        <xacro:include filename="$(find openarm_description)/urdf/ee/openarm_hand.xacro" />
-        <xacro:include filename="$(find openarm_description)/urdf/ee/openarm_hand_macro.xacro" />
-        <xacro:include filename="$(find openarm_description)/urdf/ee/openarm_hand_arguments.xacro" />
+        <xacro:include filename="${pkg_path}/urdf/ee/openarm_hand.xacro" />
+        <xacro:include filename="${pkg_path}/urdf/ee/openarm_hand_macro.xacro" />
+        <xacro:include filename="${pkg_path}/urdf/ee/openarm_hand_arguments.xacro" />
     </xacro:if>
     <xacro:property name="arm_prefix_modified" value="${'' if arm_prefix == '' else arm_prefix + '_'}" />
@@ -66,5 +66,5 @@
         kinematics_link="${body_kinematics_link}" />
         <xacro:if value="${has_head}">
-            <xacro:include filename="$(find openarm_description)/urdf/head/openarm_head.xacro" />
+            <xacro:include filename="${pkg_path}/urdf/head/openarm_head.xacro" />
             <joint name="openarm_head_mount" type="fixed">
                 <parent link="${body_link0_name}" />
@@ -120,6 +120,6 @@
                 arm_prefix="left_"
                 ee_type="${ee_type}"
-                ee_kinematics_link="${xacro.load_yaml('$(find openarm_description)/config/hand/openarm_hand/kinematics_link.yaml')}"
-                ee_inertials="${xacro.load_yaml('$(find openarm_description)/config/hand/openarm_hand/inertials.yaml')}"
+                ee_kinematics_link="${xacro.load_yaml(pkg_path + '/config/hand/openarm_hand/kinematics_link.yaml')}"
+                ee_inertials="${xacro.load_yaml(pkg_path + '/config/hand/openarm_hand/inertials.yaml')}"
                 rpy_ee="$(arg rpy_ee)"
                 xyz_ee="$(arg xyz_ee)"
@@ -133,6 +133,6 @@
                 arm_prefix="right_"
                 ee_type="${ee_type}"
-                ee_kinematics_link="${xacro.load_yaml('$(find openarm_description)/config/hand/openarm_hand/kinematics_link.yaml')}"
-                ee_inertials="${xacro.load_yaml('$(find openarm_description)/config/hand/openarm_hand/inertials.yaml')}"
+                ee_kinematics_link="${xacro.load_yaml(pkg_path + '/config/hand/openarm_hand/kinematics_link.yaml')}"
+                ee_inertials="${xacro.load_yaml(pkg_path + '/config/hand/openarm_hand/inertials.yaml')}"
                 rpy_ee="$(arg rpy_ee)"
                 xyz_ee="$(arg xyz_ee)"
@@ -147,5 +147,5 @@
                     <origin rpy="0 0 3.1416" xyz="0 0 0"/>
                     <geometry>
-                    <mesh filename="package://openarm_description/meshes/ee/rh56f1/visual/rh56f1_mount.stl" scale="0.001 0.001 0.001"/>
+                    <mesh filename="${mesh_prefix}/meshes/ee/rh56f1/visual/rh56f1_mount.stl" scale="0.001 0.001 0.001"/>
                     </geometry>
                 </visual>
@@ -167,5 +167,5 @@
                     <origin rpy="0 0 0" xyz="0 0 0"/>
                     <geometry>
-                    <mesh filename="package://openarm_description/meshes/ee/rh56f1/visual/rh56f1_mount.stl" scale="0.001 0.001 0.001"/>
+                    <mesh filename="${mesh_prefix}/meshes/ee/rh56f1/visual/rh56f1_mount.stl" scale="0.001 0.001 0.001"/>
                     </geometry>
                 </visual>
@@ -218,6 +218,6 @@
             arm_prefix="${arm_prefix_modified}"
             ee_type="${ee_type}"
-            ee_kinematics_link="${xacro.load_yaml('$(find openarm_description)/config/hand/openarm_hand/kinematics_link.yaml')}"
-            ee_inertials="${xacro.load_yaml('$(find openarm_description)/config/hand/openarm_hand/inertials.yaml')}"
+            ee_kinematics_link="${xacro.load_yaml(pkg_path + '/config/hand/openarm_hand/kinematics_link.yaml')}"
+            ee_inertials="${xacro.load_yaml(pkg_path + '/config/hand/openarm_hand/inertials.yaml')}"
             rpy_ee="$(arg rpy_ee)"
             xyz_ee="$(arg xyz_ee)"

File: urdf/robot/v10.urdf.xacro (robot description, xacro)
@@ -1,5 +1,17 @@
 <?xml version='1.0' encoding='utf-8'?>
 <robot xmlns:xacro="http://www.ros.org/wiki/xacro" name="openarm">
-  <xacro:include filename="$(find openarm_description)/urdf/robot/openarm_robot.xacro"/>
+  <xacro:arg name="pkg_path" default="" />
+  <xacro:property name="pkg_path_arg" value="$(arg pkg_path)" />
+  <!-- ROS mode (default): use $(find ...) and package:// -->
+  <xacro:if value="${pkg_path_arg == ''}">
+    <xacro:property name="pkg_path" value="$(find openarm_description)" scope="global" />
+    <xacro:property name="mesh_prefix" value="package://openarm_description" scope="global" />
+  </xacro:if>
+  <!-- Standalone mode: use absolute path and file:// -->
+  <xacro:unless value="${pkg_path_arg == ''}">
+    <xacro:property name="pkg_path" value="${pkg_path_arg}" scope="global" />
+    <xacro:property name="mesh_prefix" value="file://${pkg_path_arg}" scope="global" />
+  </xacro:unless>
+  <xacro:include filename="${pkg_path}/urdf/robot/openarm_robot.xacro"/>
   <xacro:arg name="arm_type" default="v10" />
   <xacro:arg name="body_type" default="v10" />
@@ -27,13 +39,13 @@
   arm_type="v10"
   body_type="v10"
-  joint_limits="${xacro.load_yaml('$(find openarm_description)/config//arm/v10/joint_limits.yaml')}"
-  inertials="${xacro.load_yaml('$(find openarm_description)/config/arm/v10/inertials.yaml')}"
-  kinematics="${xacro.load_yaml('$(find openarm_description)/config/arm/v10/kinematics.yaml')}"
-  kinematics_link="${xacro.load_yaml('$(find openarm_description)/config/arm/v10/kinematics_link.yaml')}"
-  kinematics_offset="${xacro.load_yaml('$(find openarm_description)/config/arm/v10/kinematics_offset.yaml')}"
-  body_inertials="${xacro.load_yaml('$(find openarm_description)/config/body/v10/inertials.yaml')}"
-  body_kinematics="${xacro.load_yaml('$(find openarm_description)/config/body/v10/kinematics.yaml')}"
-  body_kinematics_link="${xacro.load_yaml('$(find openarm_description)/config/body/v10/kinematics.yaml')}"
-  ee_kinematics_link="${xacro.load_yaml('$(find openarm_description)/config/hand/openarm_hand/kinematics_link.yaml')}"
+  joint_limits="${xacro.load_yaml(pkg_path + '/config/arm/v10/joint_limits.yaml')}"
+  inertials="${xacro.load_yaml(pkg_path + '/config/arm/v10/inertials.yaml')}"
+  kinematics="${xacro.load_yaml(pkg_path + '/config/arm/v10/kinematics.yaml')}"
+  kinematics_link="${xacro.load_yaml(pkg_path + '/config/arm/v10/kinematics_link.yaml')}"
+  kinematics_offset="${xacro.load_yaml(pkg_path + '/config/arm/v10/kinematics_offset.yaml')}"
+  body_inertials="${xacro.load_yaml(pkg_path + '/config/body/v10/inertials.yaml')}"
+  body_kinematics="${xacro.load_yaml(pkg_path + '/config/body/v10/kinematics.yaml')}"
+  body_kinematics_link="${xacro.load_yaml(pkg_path + '/config/body/v10/kinematics.yaml')}"
+  ee_kinematics_link="${xacro.load_yaml(pkg_path + '/config/hand/openarm_hand/kinematics_link.yaml')}"
   ee_type="$(arg ee_type)"
   has_head="$(arg has_head)"
