Commit message: Relative path

File: urdf/arm/openarm_arm.xacro (robot description, xacro)
@@ -1,5 +1,5 @@
 <?xml version='1.0' encoding='utf-8'?>
 <robot xmlns:xacro="http://www.ros.org/wiki/xacro" name="openarm">
-  <xacro:include filename="${pkg_path}/urdf/arm/openarm_macro.xacro" />
+  <xacro:include filename="openarm_macro.xacro" />
   <xacro:macro name="openarm_arm" params="arm_type arm_prefix:='' no_prefix:=false description_pkg:='openarm_description' connected_to:='base' xyz:='0 0 0' rpy:='0 0 0' joint_limits inertials kinematics kinematics_link kinematics_offset:=none " >
     <xacro:property name="prefix" value="${'' if no_prefix else 'openarm' + '_' + arm_prefix}" />

File: urdf/body/openarm_body.xacro (robot description, xacro)
@@ -1,5 +1,5 @@
 <?xml version="1.0" encoding="utf-8"?>
 <robot xmlns:xacro="http://www.ros.org/wiki/xacro" name="openarm_body">
-  <xacro:include filename="${pkg_path}/urdf/body/openarm_body_macro.xacro" />
+  <xacro:include filename="openarm_body_macro.xacro" />
       <xacro:macro name="openarm_body"
       params="body_type

File: urdf/robot/openarm_robot.xacro (robot description, xacro)
@@ -39,14 +39,14 @@
             "
             >
-    <xacro:include filename="${pkg_path}/urdf/arm/openarm_macro.xacro" />
-    <xacro:include filename="${pkg_path}/urdf/arm/openarm_arm.xacro" />
-    <xacro:include filename="${pkg_path}/urdf/body/openarm_body_macro.xacro" />
-    <xacro:include filename="${pkg_path}/urdf/body/openarm_body.xacro" />
-    <xacro:include filename="${pkg_path}/urdf/ros2_control/openarm.ros2_control.xacro" />
-    <xacro:include filename="${pkg_path}/urdf/ros2_control/openarm.bimanual.ros2_control.xacro" />
+    <xacro:include filename="../arm/openarm_macro.xacro" />
+    <xacro:include filename="../arm/openarm_arm.xacro" />
+    <xacro:include filename="../body/openarm_body_macro.xacro" />
+    <xacro:include filename="../body/openarm_body.xacro" />
+    <xacro:include filename="../ros2_control/openarm.ros2_control.xacro" />
+    <xacro:include filename="../ros2_control/openarm.bimanual.ros2_control.xacro" />
     <xacro:if value="${ee_type == 'openarm_hand'}">
-        <xacro:include filename="${pkg_path}/urdf/ee/openarm_hand.xacro" />
-        <xacro:include filename="${pkg_path}/urdf/ee/openarm_hand_macro.xacro" />
-        <xacro:include filename="${pkg_path}/urdf/ee/openarm_hand_arguments.xacro" />
+        <xacro:include filename="../ee/openarm_hand.xacro" />
+        <xacro:include filename="../ee/openarm_hand_macro.xacro" />
+        <xacro:include filename="../ee/openarm_hand_arguments.xacro" />
     </xacro:if>
     <xacro:property name="arm_prefix_modified" value="${'' if arm_prefix == '' else arm_prefix + '_'}" />
@@ -66,5 +66,5 @@
         kinematics_link="${body_kinematics_link}" />
         <xacro:if value="${has_head}">
-            <xacro:include filename="${pkg_path}/urdf/head/openarm_head.xacro" />
+            <xacro:include filename="../head/openarm_head.xacro" />
             <joint name="openarm_head_mount" type="fixed">
                 <parent link="${body_link0_name}" />
@@ -120,6 +120,6 @@
                 arm_prefix="left_"
                 ee_type="${ee_type}"
-                ee_kinematics_link="${xacro.load_yaml(pkg_path + '/config/hand/openarm_hand/kinematics_link.yaml')}"
-                ee_inertials="${xacro.load_yaml(pkg_path + '/config/hand/openarm_hand/inertials.yaml')}"
+                ee_kinematics_link="${xacro.load_yaml('../../config/hand/openarm_hand/kinematics_link.yaml')}"
+                ee_inertials="${xacro.load_yaml('../../config/hand/openarm_hand/inertials.yaml')}"
                 rpy_ee="$(arg rpy_ee)"
                 xyz_ee="$(arg xyz_ee)"
@@ -133,6 +133,6 @@
                 arm_prefix="right_"
                 ee_type="${ee_type}"
-                ee_kinematics_link="${xacro.load_yaml(pkg_path + '/config/hand/openarm_hand/kinematics_link.yaml')}"
-                ee_inertials="${xacro.load_yaml(pkg_path + '/config/hand/openarm_hand/inertials.yaml')}"
+                ee_kinematics_link="${xacro.load_yaml('../../config/hand/openarm_hand/kinematics_link.yaml')}"
+                ee_inertials="${xacro.load_yaml('../../config/hand/openarm_hand/inertials.yaml')}"
                 rpy_ee="$(arg rpy_ee)"
                 xyz_ee="$(arg xyz_ee)"
@@ -218,6 +218,6 @@
             arm_prefix="${arm_prefix_modified}"
             ee_type="${ee_type}"
-            ee_kinematics_link="${xacro.load_yaml(pkg_path + '/config/hand/openarm_hand/kinematics_link.yaml')}"
-            ee_inertials="${xacro.load_yaml(pkg_path + '/config/hand/openarm_hand/inertials.yaml')}"
+            ee_kinematics_link="${xacro.load_yaml('../../config/hand/openarm_hand/kinematics_link.yaml')}"
+            ee_inertials="${xacro.load_yaml('../../config/hand/openarm_hand/inertials.yaml')}"
             rpy_ee="$(arg rpy_ee)"
             xyz_ee="$(arg xyz_ee)"

File: urdf/robot/v10.urdf.xacro (robot description, xacro)
@@ -1,17 +1,14 @@
 <?xml version='1.0' encoding='utf-8'?>
 <robot xmlns:xacro="http://www.ros.org/wiki/xacro" name="openarm">
-  <xacro:arg name="pkg_path" default="" />
-  <xacro:property name="pkg_path_arg" value="$(arg pkg_path)" />
-  <!-- ROS mode (default): use $(find ...) and package:// -->
-  <xacro:if value="${pkg_path_arg == ''}">
-    <xacro:property name="pkg_path" value="$(find openarm_description)" scope="global" />
+  <xacro:arg name="standalone" default="false" />
+  <!-- ROS mode (default): use package:// for meshes -->
+  <xacro:unless value="$(arg standalone)">
     <xacro:property name="mesh_prefix" value="package://openarm_description" scope="global" />
+  </xacro:unless>
+  <!-- Standalone mode: use relative paths for meshes -->
+  <xacro:if value="$(arg standalone)">
+    <xacro:property name="mesh_prefix" value="." scope="global" />
   </xacro:if>
-  <!-- Standalone mode: use absolute path and file:// -->
-  <xacro:unless value="${pkg_path_arg == ''}">
-    <xacro:property name="pkg_path" value="${pkg_path_arg}" scope="global" />
-    <xacro:property name="mesh_prefix" value="file://${pkg_path_arg}" scope="global" />
-  </xacro:unless>
-  <xacro:include filename="${pkg_path}/urdf/robot/openarm_robot.xacro"/>
+  <xacro:include filename="openarm_robot.xacro"/>
   <xacro:arg name="arm_type" default="v10" />
   <xacro:arg name="body_type" default="v10" />
@@ -39,13 +36,13 @@
   arm_type="v10"
   body_type="v10"
-  joint_limits="${xacro.load_yaml(pkg_path + '/config/arm/v10/joint_limits.yaml')}"
-  inertials="${xacro.load_yaml(pkg_path + '/config/arm/v10/inertials.yaml')}"
-  kinematics="${xacro.load_yaml(pkg_path + '/config/arm/v10/kinematics.yaml')}"
-  kinematics_link="${xacro.load_yaml(pkg_path + '/config/arm/v10/kinematics_link.yaml')}"
-  kinematics_offset="${xacro.load_yaml(pkg_path + '/config/arm/v10/kinematics_offset.yaml')}"
-  body_inertials="${xacro.load_yaml(pkg_path + '/config/body/v10/inertials.yaml')}"
-  body_kinematics="${xacro.load_yaml(pkg_path + '/config/body/v10/kinematics.yaml')}"
-  body_kinematics_link="${xacro.load_yaml(pkg_path + '/config/body/v10/kinematics.yaml')}"
-  ee_kinematics_link="${xacro.load_yaml(pkg_path + '/config/hand/openarm_hand/kinematics_link.yaml')}"
+  joint_limits="${xacro.load_yaml('../../config/arm/v10/joint_limits.yaml')}"
+  inertials="${xacro.load_yaml('../../config/arm/v10/inertials.yaml')}"
+  kinematics="${xacro.load_yaml('../../config/arm/v10/kinematics.yaml')}"
+  kinematics_link="${xacro.load_yaml('../../config/arm/v10/kinematics_link.yaml')}"
+  kinematics_offset="${xacro.load_yaml('../../config/arm/v10/kinematics_offset.yaml')}"
+  body_inertials="${xacro.load_yaml('../../config/body/v10/inertials.yaml')}"
+  body_kinematics="${xacro.load_yaml('../../config/body/v10/kinematics.yaml')}"
+  body_kinematics_link="${xacro.load_yaml('../../config/body/v10/kinematics.yaml')}"
+  ee_kinematics_link="${xacro.load_yaml('../../config/hand/openarm_hand/kinematics_link.yaml')}"
   ee_type="$(arg ee_type)"
   has_head="$(arg has_head)"
