Commit message: Hand file directory

File: inspire_hand_description/RH56F1/left/urdf/RH56F1_L.xacro (robot description, xacro)
@@ -27,5 +27,5 @@
       <geometry>
         <mesh
-          filename="package://inspire_hand_description/RH56F1/left/meshes/base_link.STL" />
+          filename="${hand_mesh_prefix}/RH56F1/left/meshes/base_link.STL" />
       </geometry>
       <material
@@ -41,5 +41,5 @@
       <geometry>
         <mesh
-          filename="package://inspire_hand_description/RH56F1/left/meshes/base_link.STL" />
+          filename="${hand_mesh_prefix}/RH56F1/left/meshes/base_link.STL" />
       </geometry>
     </collision>
@@ -67,5 +67,5 @@
       <geometry>
         <mesh
-          filename="package://inspire_hand_description/RH56F1/left/meshes/left_thumb_1.STL" />
+          filename="${hand_mesh_prefix}/RH56F1/left/meshes/left_thumb_1.STL" />
       </geometry>
       <material
@@ -81,5 +81,5 @@
       <geometry>
         <mesh
-          filename="package://inspire_hand_description/RH56F1/left/meshes/left_thumb_1.STL" />
+          filename="${hand_mesh_prefix}/RH56F1/left/meshes/left_thumb_1.STL" />
       </geometry>
     </collision>
@@ -125,19 +125,19 @@
       <geometry>
         <mesh
-          filename="package://inspire_hand_description/RH56F1/left/meshes/left_thumb_2.STL" />
-      </geometry>
-      <material
-        name="">
-        <color
-          rgba="0.25 0.25 0.25 1" />
-      </material>
-    </visual>
-    <collision>
-      <origin
-        xyz="0 0 0"
-        rpy="0 0 0" />
-      <geometry>
-        <mesh
-          filename="package://inspire_hand_description/RH56F1/left/meshes/left_thumb_2.STL" />
+          filename="${hand_mesh_prefix}/RH56F1/left/meshes/left_thumb_2.STL" />
+      </geometry>
+      <material
+        name="">
+        <color
+          rgba="0.25 0.25 0.25 1" />
+      </material>
+    </visual>
+    <collision>
+      <origin
+        xyz="0 0 0"
+        rpy="0 0 0" />
+      <geometry>
+        <mesh
+          filename="${hand_mesh_prefix}/RH56F1/left/meshes/left_thumb_2.STL" />
       </geometry>
     </collision>
@@ -183,19 +183,19 @@
       <geometry>
         <mesh
-          filename="package://inspire_hand_description/RH56F1/left/meshes/left_thumb_3.STL" />
-      </geometry>
-      <material
-        name="">
-        <color
-          rgba="0.25 0.25 0.25 1" />
-      </material>
-    </visual>
-    <collision>
-      <origin
-        xyz="0 0 0"
-        rpy="0 0 0" />
-      <geometry>
-        <mesh
-          filename="package://inspire_hand_description/RH56F1/left/meshes/left_thumb_3.STL" />
+          filename="${hand_mesh_prefix}/RH56F1/left/meshes/left_thumb_3.STL" />
+      </geometry>
+      <material
+        name="">
+        <color
+          rgba="0.25 0.25 0.25 1" />
+      </material>
+    </visual>
+    <collision>
+      <origin
+        xyz="0 0 0"
+        rpy="0 0 0" />
+      <geometry>
+        <mesh
+          filename="${hand_mesh_prefix}/RH56F1/left/meshes/left_thumb_3.STL" />
       </geometry>
     </collision>
@@ -245,19 +245,19 @@
       <geometry>
         <mesh
-          filename="package://inspire_hand_description/RH56F1/left/meshes/left_thumb_4.STL" />
-      </geometry>
-      <material
-        name="">
-        <color
-          rgba="0.25 0.25 0.25 1" />
-      </material>
-    </visual>
-    <collision>
-      <origin
-        xyz="0 0 0"
-        rpy="0 0 0" />
-      <geometry>
-        <mesh
-          filename="package://inspire_hand_description/RH56F1/left/meshes/left_thumb_4.STL" />
+          filename="${hand_mesh_prefix}/RH56F1/left/meshes/left_thumb_4.STL" />
+      </geometry>
+      <material
+        name="">
+        <color
+          rgba="0.25 0.25 0.25 1" />
+      </material>
+    </visual>
+    <collision>
+      <origin
+        xyz="0 0 0"
+        rpy="0 0 0" />
+      <geometry>
+        <mesh
+          filename="${hand_mesh_prefix}/RH56F1/left/meshes/left_thumb_4.STL" />
       </geometry>
     </collision>
@@ -307,19 +307,19 @@
       <geometry>
         <mesh
-          filename="package://inspire_hand_description/RH56F1/left/meshes/thumb_force_sensor.STL" />
-      </geometry>
-      <material
-        name="">
-        <color
-          rgba="0.25 0.25 0.25 1" />
-      </material>
-    </visual>
-    <collision>
-      <origin
-        xyz="0 0 0"
-        rpy="0 0 0" />
-      <geometry>
-        <mesh
-          filename="package://inspire_hand_description/RH56F1/left/meshes/thumb_force_sensor.STL" />
+          filename="${hand_mesh_prefix}/RH56F1/left/meshes/thumb_force_sensor.STL" />
+      </geometry>
+      <material
+        name="">
+        <color
+          rgba="0.25 0.25 0.25 1" />
+      </material>
+    </visual>
+    <collision>
+      <origin
+        xyz="0 0 0"
+        rpy="0 0 0" />
+      <geometry>
+        <mesh
+          filename="${hand_mesh_prefix}/RH56F1/left/meshes/thumb_force_sensor.STL" />
       </geometry>
     </collision>
@@ -360,19 +360,19 @@
       <geometry>
         <mesh
-          filename="package://inspire_hand_description/RH56F1/left/meshes/thumb_tip.STL" />
-      </geometry>
-      <material
-        name="">
-        <color
-          rgba="0.25 0.25 0.25 1" />
-      </material>
-    </visual>
-    <collision>
-      <origin
-        xyz="0 0 0"
-        rpy="0 0 0" />
-      <geometry>
-        <mesh
-          filename="package://inspire_hand_description/RH56F1/left/meshes/thumb_tip.STL" />
+          filename="${hand_mesh_prefix}/RH56F1/left/meshes/thumb_tip.STL" />
+      </geometry>
+      <material
+        name="">
+        <color
+          rgba="0.25 0.25 0.25 1" />
+      </material>
+    </visual>
+    <collision>
+      <origin
+        xyz="0 0 0"
+        rpy="0 0 0" />
+      <geometry>
+        <mesh
+          filename="${hand_mesh_prefix}/RH56F1/left/meshes/thumb_tip.STL" />
       </geometry>
     </collision>
@@ -413,19 +413,19 @@
       <geometry>
         <mesh
-          filename="package://inspire_hand_description/RH56F1/left/meshes/left_index_1.STL" />
-      </geometry>
-      <material
-        name="">
-        <color
-          rgba="0.25 0.25 0.25 1" />
-      </material>
-    </visual>
-    <collision>
-      <origin
-        xyz="0 0 0"
-        rpy="0 0 0" />
-      <geometry>
-        <mesh
-          filename="package://inspire_hand_description/RH56F1/left/meshes/left_index_1.STL" />
+          filename="${hand_mesh_prefix}/RH56F1/left/meshes/left_index_1.STL" />
+      </geometry>
+      <material
+        name="">
+        <color
+          rgba="0.25 0.25 0.25 1" />
+      </material>
+    </visual>
+    <collision>
+      <origin
+        xyz="0 0 0"
+        rpy="0 0 0" />
+      <geometry>
+        <mesh
+          filename="${hand_mesh_prefix}/RH56F1/left/meshes/left_index_1.STL" />
       </geometry>
     </collision>
@@ -471,19 +471,19 @@
       <geometry>
         <mesh
-          filename="package://inspire_hand_description/RH56F1/left/meshes/left_index_2.STL" />
-      </geometry>
-      <material
-        name="">
-        <color
-          rgba="0.25 0.25 0.25 1" />
-      </material>
-    </visual>
-    <collision>
-      <origin
-        xyz="0 0 0"
-        rpy="0 0 0" />
-      <geometry>
-        <mesh
-          filename="package://inspire_hand_description/RH56F1/left/meshes/left_index_2.STL" />
+          filename="${hand_mesh_prefix}/RH56F1/left/meshes/left_index_2.STL" />
+      </geometry>
+      <material
+        name="">
+        <color
+          rgba="0.25 0.25 0.25 1" />
+      </material>
+    </visual>
+    <collision>
+      <origin
+        xyz="0 0 0"
+        rpy="0 0 0" />
+      <geometry>
+        <mesh
+          filename="${hand_mesh_prefix}/RH56F1/left/meshes/left_index_2.STL" />
       </geometry>
     </collision>
@@ -533,19 +533,19 @@
       <geometry>
         <mesh
-          filename="package://inspire_hand_description/RH56F1/left/meshes/index_force_sensor.STL" />
-      </geometry>
-      <material
-        name="">
-        <color
-          rgba="0.25 0.25 0.25 1" />
-      </material>
-    </visual>
-    <collision>
-      <origin
-        xyz="0 0 0"
-        rpy="0 0 0" />
-      <geometry>
-        <mesh
-          filename="package://inspire_hand_description/RH56F1/left/meshes/index_force_sensor.STL" />
+          filename="${hand_mesh_prefix}/RH56F1/left/meshes/index_force_sensor.STL" />
+      </geometry>
+      <material
+        name="">
+        <color
+          rgba="0.25 0.25 0.25 1" />
+      </material>
+    </visual>
+    <collision>
+      <origin
+        xyz="0 0 0"
+        rpy="0 0 0" />
+      <geometry>
+        <mesh
+          filename="${hand_mesh_prefix}/RH56F1/left/meshes/index_force_sensor.STL" />
       </geometry>
     </collision>
@@ -586,19 +586,19 @@
       <geometry>
         <mesh
-          filename="package://inspire_hand_description/RH56F1/left/meshes/index_tip.STL" />
-      </geometry>
-      <material
-        name="">
-        <color
-          rgba="0.25 0.25 0.25 1" />
-      </material>
-    </visual>
-    <collision>
-      <origin
-        xyz="0 0 0"
-        rpy="0 0 0" />
-      <geometry>
-        <mesh
-          filename="package://inspire_hand_description/RH56F1/left/meshes/index_tip.STL" />
+          filename="${hand_mesh_prefix}/RH56F1/left/meshes/index_tip.STL" />
+      </geometry>
+      <material
+        name="">
+        <color
+          rgba="0.25 0.25 0.25 1" />
+      </material>
+    </visual>
+    <collision>
+      <origin
+        xyz="0 0 0"
+        rpy="0 0 0" />
+      <geometry>
+        <mesh
+          filename="${hand_mesh_prefix}/RH56F1/left/meshes/index_tip.STL" />
       </geometry>
     </collision>
@@ -639,19 +639,19 @@
       <geometry>
         <mesh
-          filename="package://inspire_hand_description/RH56F1/left/meshes/left_middle_1.STL" />
-      </geometry>
-      <material
-        name="">
-        <color
-          rgba="0.25 0.25 0.25 1" />
-      </material>
-    </visual>
-    <collision>
-      <origin
-        xyz="0 0 0"
-        rpy="0 0 0" />
-      <geometry>
-        <mesh
-          filename="package://inspire_hand_description/RH56F1/left/meshes/left_middle_1.STL" />
+          filename="${hand_mesh_prefix}/RH56F1/left/meshes/left_middle_1.STL" />
+      </geometry>
+      <material
+        name="">
+        <color
+          rgba="0.25 0.25 0.25 1" />
+      </material>
+    </visual>
+    <collision>
+      <origin
+        xyz="0 0 0"
+        rpy="0 0 0" />
+      <geometry>
+        <mesh
+          filename="${hand_mesh_prefix}/RH56F1/left/meshes/left_middle_1.STL" />
       </geometry>
     </collision>
@@ -697,19 +697,19 @@
       <geometry>
         <mesh
-          filename="package://inspire_hand_description/RH56F1/left/meshes/left_middle_2.STL" />
-      </geometry>
-      <material
-        name="">
-        <color
-          rgba="0.25 0.25 0.25 1" />
-      </material>
-    </visual>
-    <collision>
-      <origin
-        xyz="0 0 0"
-        rpy="0 0 0" />
-      <geometry>
-        <mesh
-          filename="package://inspire_hand_description/RH56F1/left/meshes/left_middle_2.STL" />
+          filename="${hand_mesh_prefix}/RH56F1/left/meshes/left_middle_2.STL" />
+      </geometry>
+      <material
+        name="">
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
File: inspire_hand_description/RH56F1/right/urdf/RH56F1_R.xacro (robot description, xacro)
@@ -27,5 +27,5 @@
       <geometry>
         <mesh
-          filename="package://inspire_hand_description/RH56F1/right/meshes/base_link.STL" />
+          filename="${hand_mesh_prefix}/RH56F1/right/meshes/base_link.STL" />
       </geometry>
       <material
@@ -41,5 +41,5 @@
       <geometry>
         <mesh
-          filename="package://inspire_hand_description/RH56F1/right/meshes/base_link.STL" />
+          filename="${hand_mesh_prefix}/RH56F1/right/meshes/base_link.STL" />
       </geometry>
     </collision>
@@ -67,5 +67,5 @@
       <geometry>
         <mesh
-          filename="package://inspire_hand_description/RH56F1/right/meshes/plam_1.STL" />
+          filename="${hand_mesh_prefix}/RH56F1/right/meshes/plam_1.STL" />
       </geometry>
       <material
@@ -81,5 +81,5 @@
       <geometry>
         <mesh
-          filename="package://inspire_hand_description/RH56F1/right/meshes/plam_1.STL" />
+          filename="${hand_mesh_prefix}/RH56F1/right/meshes/plam_1.STL" />
       </geometry>
     </collision>
@@ -120,19 +120,19 @@
       <geometry>
         <mesh
-          filename="package://inspire_hand_description/RH56F1/right/meshes/plam_2.STL" />
-      </geometry>
-      <material
-        name="">
-        <color
-          rgba="0.25 0.25 0.25 1" />
-      </material>
-    </visual>
-    <collision>
-      <origin
-        xyz="0 0 0"
-        rpy="0 0 0" />
-      <geometry>
-        <mesh
-          filename="package://inspire_hand_description/RH56F1/right/meshes/plam_2.STL" />
+          filename="${hand_mesh_prefix}/RH56F1/right/meshes/plam_2.STL" />
+      </geometry>
+      <material
+        name="">
+        <color
+          rgba="0.25 0.25 0.25 1" />
+      </material>
+    </visual>
+    <collision>
+      <origin
+        xyz="0 0 0"
+        rpy="0 0 0" />
+      <geometry>
+        <mesh
+          filename="${hand_mesh_prefix}/RH56F1/right/meshes/plam_2.STL" />
       </geometry>
     </collision>
@@ -173,5 +173,5 @@
       <geometry>
         <mesh
-          filename="package://inspire_hand_description/RH56F1/right/meshes/plam_3.STL" />
+          filename="${hand_mesh_prefix}/RH56F1/right/meshes/plam_3.STL" />
       </geometry>
       <material
@@ -187,5 +187,5 @@
       <geometry>
         <mesh
-          filename="package://inspire_hand_description/RH56F1/right/meshes/plam_3.STL" />
+          filename="${hand_mesh_prefix}/RH56F1/right/meshes/plam_3.STL" />
       </geometry>
     </collision>
@@ -226,5 +226,5 @@
       <geometry>
         <mesh
-          filename="package://inspire_hand_description/RH56F1/right/meshes/plam_force_sensor.STL" />
+          filename="${hand_mesh_prefix}/RH56F1/right/meshes/plam_force_sensor.STL" />
       </geometry>
       <material
@@ -240,5 +240,5 @@
       <geometry>
         <mesh
-          filename="package://inspire_hand_description/RH56F1/right/meshes/plam_force_sensor.STL" />
+          filename="${hand_mesh_prefix}/RH56F1/right/meshes/plam_force_sensor.STL" />
       </geometry>
     </collision>
@@ -279,5 +279,5 @@
       <geometry>
         <mesh
-          filename="package://inspire_hand_description/RH56F1/right/meshes/right_thumb_1.STL" />
+          filename="${hand_mesh_prefix}/RH56F1/right/meshes/right_thumb_1.STL" />
       </geometry>
       <material
@@ -293,5 +293,5 @@
       <geometry>
         <mesh
-          filename="package://inspire_hand_description/RH56F1/right/meshes/right_thumb_1.STL" />
+          filename="${hand_mesh_prefix}/RH56F1/right/meshes/right_thumb_1.STL" />
       </geometry>
     </collision>
@@ -337,19 +337,19 @@
       <geometry>
         <mesh
-          filename="package://inspire_hand_description/RH56F1/right/meshes/right_thumb_2.STL" />
-      </geometry>
-      <material
-        name="">
-        <color
-          rgba="0.25 0.25 0.25 1" />
-      </material>
-    </visual>
-    <collision>
-      <origin
-        xyz="0 0 0"
-        rpy="0 0 0" />
-      <geometry>
-        <mesh
-          filename="package://inspire_hand_description/RH56F1/right/meshes/right_thumb_2.STL" />
+          filename="${hand_mesh_prefix}/RH56F1/right/meshes/right_thumb_2.STL" />
+      </geometry>
+      <material
+        name="">
+        <color
+          rgba="0.25 0.25 0.25 1" />
+      </material>
+    </visual>
+    <collision>
+      <origin
+        xyz="0 0 0"
+        rpy="0 0 0" />
+      <geometry>
+        <mesh
+          filename="${hand_mesh_prefix}/RH56F1/right/meshes/right_thumb_2.STL" />
       </geometry>
     </collision>
@@ -395,19 +395,19 @@
       <geometry>
         <mesh
-          filename="package://inspire_hand_description/RH56F1/right/meshes/right_thumb_3.STL" />
-      </geometry>
-      <material
-        name="">
-        <color
-          rgba="0.25 0.25 0.25 1" />
-      </material>
-    </visual>
-    <collision>
-      <origin
-        xyz="0 0 0"
-        rpy="0 0 0" />
-      <geometry>
-        <mesh
-          filename="package://inspire_hand_description/RH56F1/right/meshes/right_thumb_3.STL" />
+          filename="${hand_mesh_prefix}/RH56F1/right/meshes/right_thumb_3.STL" />
+      </geometry>
+      <material
+        name="">
+        <color
+          rgba="0.25 0.25 0.25 1" />
+      </material>
+    </visual>
+    <collision>
+      <origin
+        xyz="0 0 0"
+        rpy="0 0 0" />
+      <geometry>
+        <mesh
+          filename="${hand_mesh_prefix}/RH56F1/right/meshes/right_thumb_3.STL" />
       </geometry>
     </collision>
@@ -457,19 +457,19 @@
       <geometry>
         <mesh
-          filename="package://inspire_hand_description/RH56F1/right/meshes/right_thumb_4.STL" />
-      </geometry>
-      <material
-        name="">
-        <color
-          rgba="0.25 0.25 0.25 1" />
-      </material>
-    </visual>
-    <collision>
-      <origin
-        xyz="0 0 0"
-        rpy="0 0 0" />
-      <geometry>
-        <mesh
-          filename="package://inspire_hand_description/RH56F1/right/meshes/right_thumb_4.STL" />
+          filename="${hand_mesh_prefix}/RH56F1/right/meshes/right_thumb_4.STL" />
+      </geometry>
+      <material
+        name="">
+        <color
+          rgba="0.25 0.25 0.25 1" />
+      </material>
+    </visual>
+    <collision>
+      <origin
+        xyz="0 0 0"
+        rpy="0 0 0" />
+      <geometry>
+        <mesh
+          filename="${hand_mesh_prefix}/RH56F1/right/meshes/right_thumb_4.STL" />
       </geometry>
     </collision>
@@ -519,19 +519,19 @@
       <geometry>
         <mesh
-          filename="package://inspire_hand_description/RH56F1/right/meshes/thumb_force_sensor.STL" />
-      </geometry>
-      <material
-        name="">
-        <color
-          rgba="0.25 0.25 0.25 1" />
-      </material>
-    </visual>
-    <collision>
-      <origin
-        xyz="0 0 0"
-        rpy="0 0 0" />
-      <geometry>
-        <mesh
-          filename="package://inspire_hand_description/RH56F1/right/meshes/thumb_force_sensor.STL" />
+          filename="${hand_mesh_prefix}/RH56F1/right/meshes/thumb_force_sensor.STL" />
+      </geometry>
+      <material
+        name="">
+        <color
+          rgba="0.25 0.25 0.25 1" />
+      </material>
+    </visual>
+    <collision>
+      <origin
+        xyz="0 0 0"
+        rpy="0 0 0" />
+      <geometry>
+        <mesh
+          filename="${hand_mesh_prefix}/RH56F1/right/meshes/thumb_force_sensor.STL" />
       </geometry>
     </collision>
@@ -572,19 +572,19 @@
       <geometry>
         <mesh
-          filename="package://inspire_hand_description/RH56F1/right/meshes/thumb_tip.STL" />
-      </geometry>
-      <material
-        name="">
-        <color
-          rgba="0.25 0.25 0.25 1" />
-      </material>
-    </visual>
-    <collision>
-      <origin
-        xyz="0 0 0"
-        rpy="0 0 0" />
-      <geometry>
-        <mesh
-          filename="package://inspire_hand_description/RH56F1/right/meshes/thumb_tip.STL" />
+          filename="${hand_mesh_prefix}/RH56F1/right/meshes/thumb_tip.STL" />
+      </geometry>
+      <material
+        name="">
+        <color
+          rgba="0.25 0.25 0.25 1" />
+      </material>
+    </visual>
+    <collision>
+      <origin
+        xyz="0 0 0"
+        rpy="0 0 0" />
+      <geometry>
+        <mesh
+          filename="${hand_mesh_prefix}/RH56F1/right/meshes/thumb_tip.STL" />
       </geometry>
     </collision>
@@ -625,19 +625,19 @@
       <geometry>
         <mesh
-          filename="package://inspire_hand_description/RH56F1/right/meshes/right_index_1.STL" />
-      </geometry>
-      <material
-        name="">
-        <color
-          rgba="0.25 0.25 0.25 1" />
-      </material>
-    </visual>
-    <collision>
-      <origin
-        xyz="0 0 0"
-        rpy="0 0 0" />
-      <geometry>
-        <mesh
-          filename="package://inspire_hand_description/RH56F1/right/meshes/right_index_1.STL" />
+          filename="${hand_mesh_prefix}/RH56F1/right/meshes/right_index_1.STL" />
+      </geometry>
+      <material
+        name="">
+        <color
+          rgba="0.25 0.25 0.25 1" />
+      </material>
+    </visual>
+    <collision>
+      <origin
+        xyz="0 0 0"
+        rpy="0 0 0" />
+      <geometry>
+        <mesh
+          filename="${hand_mesh_prefix}/RH56F1/right/meshes/right_index_1.STL" />
       </geometry>
     </collision>
@@ -683,19 +683,19 @@
       <geometry>
         <mesh
-          filename="package://inspire_hand_description/RH56F1/right/meshes/right_index_2.STL" />
-      </geometry>
-      <material
-        name="">
-        <color
-          rgba="0.25 0.25 0.25 1" />
-      </material>
-    </visual>
-    <collision>
-      <origin
-        xyz="0 0 0"
-        rpy="0 0 0" />
-      <geometry>
-        <mesh
-          filename="package://inspire_hand_description/RH56F1/right/meshes/right_index_2.STL" />
+          filename="${hand_mesh_prefix}/RH56F1/right/meshes/right_index_2.STL" />
+      </geometry>
+      <material
+        name="">
+        <color
+          rgba="0.25 0.25 0.25 1" />
+      </material>
+    </visual>
+    <collision>
+      <origin
+        xyz="0 0 0"
+        rpy="0 0 0" />
+      <geometry>
+        <mesh
+          filename="${hand_mesh_prefix}/RH56F1/right/meshes/right_index_2.STL" />
       </geometry>
     </collision>
@@ -745,19 +745,19 @@
       <geometry>
         <mesh
-          filename="package://inspire_hand_description/RH56F1/right/meshes/index_force_sensor.STL" />
-      </geometry>
-      <material
-        name="">
-        <color
-          rgba="0.25 0.25 0.25 1" />
-      </material>
-    </visual>
-    <collision>
-      <origin
-        xyz="0 0 0"
-        rpy="0 0 0" />
-      <geometry>
-        <mesh
-          filename="package://inspire_hand_description/RH56F1/right/meshes/index_force_sensor.STL" />
+          filename="${hand_mesh_prefix}/RH56F1/right/meshes/index_force_sensor.STL" />
+      </geometry>
+      <material
+        name="">
+        <color
+          rgba="0.25 0.25 0.25 1" />
+      </material>
+    </visual>
+    <collision>
+      <origin
+        xyz="0 0 0"
+        rpy="0 0 0" />
+      <geometry>
+        <mesh
+          filename="${hand_mesh_prefix}/RH56F1/right/meshes/index_force_sensor.STL" />
       </geometry>
     </collision>
@@ -798,19 +798,19 @@
       <geometry>
         <mesh
-          filename="package://inspire_hand_description/RH56F1/right/meshes/index_tip.STL" />
-      </geometry>
-      <material
-        name="">
-        <color
-          rgba="0.25 0.25 0.25 1" />
-      </material>
-    </visual>
-    <collision>
-      <origin
-        xyz="0 0 0"
-        rpy="0 0 0" />
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