Commit message: Hand file directory

File: urdf/robot/openarm_robot.xacro (robot description, xacro)
@@ -151,5 +151,5 @@
                 </visual>
             </link>
-            <xacro:include filename="$(find inspire_hand_description)/RH56F1/left/urdf/RH56F1_L.xacro" />
+            <xacro:include filename="${hand_include_prefix}/RH56F1/left/urdf/RH56F1_L.xacro" />
             <xacro:RH56F1_L />
             <joint name="left_arm_to_mount" type="fixed">
@@ -171,5 +171,5 @@
                 </visual>
             </link>
-            <xacro:include filename="$(find inspire_hand_description)/RH56F1/right/urdf/RH56F1_R.xacro" />
+            <xacro:include filename="${hand_include_prefix}/RH56F1/right/urdf/RH56F1_R.xacro" />
             <xacro:RH56F1_R />
             <joint name="right_arm_to_mount" type="fixed">

File: urdf/robot/v10.urdf.xacro (robot description, xacro)
@@ -5,8 +5,12 @@
   <xacro:unless value="$(arg standalone)">
     <xacro:property name="mesh_prefix" value="package://openarm_description" scope="global" />
+    <xacro:property name="hand_mesh_prefix" value="package://inspire_hand_description" scope="global" />
+    <xacro:property name="hand_include_prefix" value="$(find inspire_hand_description)" scope="global" />
   </xacro:unless>
-  <!-- Standalone mode: use relative paths for meshes -->
+  <!-- Standalone mode: use relative paths -->
   <xacro:if value="$(arg standalone)">
     <xacro:property name="mesh_prefix" value="." scope="global" />
+    <xacro:property name="hand_mesh_prefix" value="./inspire_hand_description" scope="global" />
+    <xacro:property name="hand_include_prefix" value="../../inspire_hand_description" scope="global" />
   </xacro:if>
   <xacro:include filename="openarm_robot.xacro"/>
